File: hw/TinyG3DPrinterController.brd (EAGLE design)
At the start: 61 x 62 mm, 39 parts, among them CON5 MOLEX-53261-0671, IC1 MEGA164P, IC2 LM4040C41IDBZR, Q1 14.7456 MHz, T1 IRLML5203TRPBF, T2 STP55NF06L, T3 STP55NF06L, T4 STP55NF06L

Commit message: Adapted sch and brd files
Parts:
- added JP1: (no value), pinhead:1X04
- added JP2: (no value), pinhead:2X03
- added JP3: (no value), pinhead:2X05
- added JP4: (no value), pinhead:2X04
- added JP5: (no value), pinhead:1X03
- added LED3: (no value), led:CHIP-LED0805
- added R14, R15: 4k7, rcl:R0603
- added R16: 470R, rcl:R0603
- Q1: device crystal:HC49UP -> SchlegelArmin:CRYSTAL_2P_5MMX3.2MM
- moved R11 8.81 mm to (10.7, 20.1), flipped to the top, turned to 180 degrees
- moved IC2 6.60 mm to (45.0, 23.2), turned to 270 degrees
- moved C3 5.38 mm to (49.1, 31.4), turned to 270 degrees
- moved R10 4.47 mm to (30.0, 40.0), turned to 270 degrees
- moved R25 4.47 mm to (56.0, 40.0), turned to 270 degrees
- moved R6 4.47 mm to (43.0, 40.0), turned to 270 degrees
- moved C2 2.67 mm to (16.0, 20.8)
- moved C1 1.52 mm to (16.0, 24.4)
- moved R7 1.28 mm to (26.8, 37.0), turned to 0 degrees
- moved R4 1.24 mm to (39.9, 36.9), turned to 0 degrees
- moved R9 1.13 mm to (52.8, 36.8), turned to 0 degrees
- moved X3 0.80 mm to (34.0, 56.2)
- moved Q1 0.60 mm to (19.0, 22.6), turned to 270 degrees
- moved R12 0.56 mm to (39.1, 23.6)
Connections:
- new net ADC_REF_EXT: IC2.1, JP5.3, R12.1
- new net AVR_CS0: IC1.43, JP2.3
- new net AVR_CS1: IC1.44, JP3.7
- new net AVR_IO0: IC1.35, JP3.3
- new net AVR_IO1: IC1.34, JP3.4
- new net AVR_IO2: IC1.33, JP3.1
- new net AVR_IO3: IC1.32, JP3.2
- new net AVR_IO4: IC1.21, JP4.1
- new net AVR_IO5: IC1.22, JP4.2
- new net AVR_IO6: IC1.23, JP4.3
- new net AVR_IO7: IC1.24, JP4.4
- new net AVR_IO8: IC1.25, JP4.5
- new net AVR_IO9: IC1.26, JP4.6
- new net AVR_SCL: IC1.19, JP1.2, R14.1
- new net AVR_SDA: IC1.20, JP1.3, R15.1
- new net N$12: LED3.C, R16.1
- net +5V: now also JP1.1, JP2.1, JP3.5, JP4.7, JP5.1, R14.2, R15.2, R16.2
- net AVR_!RESET: no longer S1.1
- net AVR_AREF: now also JP5.2; no longer IC2.1, R12.1
- net AVR_MISO: now also JP2.6, JP3.10
- net AVR_MOSI: now also JP2.2, JP3.6
- net AVR_SCK: now also JP2.4, JP3.8
- net GND: now also JP1.4, JP2.5, JP3.9, JP4.8, LED3.A; no longer S1.3
- net N$1: now also Q1.P$2; no longer Q1.2
- net N$2: now also Q1.P$1; no longer Q1.1
Routing:
- net +5V: track 124.0 -> 180.3 mm, vias 7 -> 8
- net AVR_IO0: track 0.00 -> 28.8 mm, vias 0 -> 1
- net +24V: track 140.3 -> 114.4 mm
- net AVR_IO1: track 0.00 -> 25.4 mm, vias 0 -> 1
- net AVR_IO8: track 0.00 -> 23.1 mm
- net AVR_IO3: track 0.00 -> 22.9 mm, vias 0 -> 1
- net AVR_IO9: track 0.00 -> 21.7 mm
- net AVR_IO2: track 0.00 -> 20.8 mm, vias 0 -> 1
- net AVR_CS0: track 0.00 -> 20.5 mm
- net AVR_IO6: track 0.00 -> 19.6 mm
- net AVR_CS1: track 0.00 -> 18.5 mm
- net AVR_IO7: track 0.00 -> 18.4 mm
- net AVR_IO4: track 0.00 -> 17.9 mm
- net AVR_!RESET: track 55.5 -> 39.9 mm
- net AVR_IO5: track 0.00 -> 15.0 mm
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Other:
- board text added: "- + 24V"
- board text added: "17.07.2016"
- board text added: "Armin Schlegel"
- board text added: "FAN"
- board text added: "Heatbed"
- board text added: "Hotend"
- board text added: "I2C"
- board text added: "Thermo Heatbed"
- board text added: "Thermo Hotend"
- board text added: "TinyG Controller 3D Printer Cape V1"
