File: hw/TinyG3DPrinterController.sch (EAGLE design)
At the start: 39 parts, among them CON5 MOLEX-53261-0671, IC1 MEGA164P, IC2 LM4040C41IDBZR, Q1 14.7456 MHz, T1 IRLML5203TRPBF, T2 STP55NF06L, T3 STP55NF06L, T4 STP55NF06L

Commit message: Adapted sch and brd files
Parts:
- added JP1: (no value), pinhead:PINHD-1X4
- added JP2: (no value), pinhead:PINHD-2X3
- added JP3: (no value), pinhead:PINHD-2X5
- added JP4: (no value), pinhead:PINHD-2X4
- added JP5: (no value), pinhead:PINHD-1X3
- added LED3: (no value), led:LEDCHIP-LED0805
- added R14, R15: 4k7, rcl:R-EU_R0603
- added R16: 470R, rcl:R-EU_R0603
- Q1: device crystal:CRYSTALHC49UP -> SchlegelArmin:7A-14.7456MAAJ-T-SMD_CRYSTAL
Connections:
- new net ADC_REF_EXT: IC2.1, JP5.3, R12.1
- new net AVR_CS0: IC1.(OC0A/AIN1/PCINT11)PB3, JP2.3
- new net AVR_CS1: IC1.(OC0B/!SS!/PCINT12)PB4, JP3.7
- new net AVR_IO0: IC1.(ADC2/PCINT2)PA2, JP3.3
- new net AVR_IO1: IC1.(ADC3/PCINT3)PA3, JP3.4
- new net AVR_IO2: IC1.(ADC4/PCINT4)PA4, JP3.1
- new net AVR_IO3: IC1.(ADC5/PCINT5)PA5, JP3.2
- new net AVR_IO4: IC1.(TCK/PCINT18)PC2, JP4.1
- new net AVR_IO5: IC1.(TMS/PCINT19)PC3, JP4.2
- new net AVR_IO6: IC1.(TDO/PCINT20)PC4, JP4.3
- new net AVR_IO7: IC1.(TDI/PCINT21)PC5, JP4.4
- new net AVR_IO8: IC1.(TOSC1/PCINT22)PC6, JP4.5
- new net AVR_IO9: IC1.(TOSC2/PCINT23)PC7, JP4.6
- new net AVR_SCL: IC1.(SCL/PCINT16)PC0, JP1.2, R14.1
- new net AVR_SDA: IC1.(SDA/PCINT17)PC1, JP1.3, R15.1
- new net N$12: LED3.C, R16.1
- net +5V: now also JP1.1, JP2.1, JP3.5, JP4.7, JP5.1, R14.2, R15.2, R16.2
- net AVR_!RESET: no longer S1.S
- net AVR_AREF: now also JP5.2; no longer IC2.1, R12.1
- net AVR_MISO: now also JP2.6, JP3.10
- net AVR_MOSI: now also JP2.2, JP3.6
- net AVR_SCK: now also JP2.4, JP3.8
- net GND: now also JP1.4, JP2.5, JP3.9, JP4.8, LED3.A; no longer S1.P
